File: Eletronica/Kicad/HUA.sch (KiCad schematic (older format))
At the start: 83 parts

Commit message: EDIT: NODEMCU as a replacement for arduino (V2)
Parts:
- removed C? (x2): 100p, Capacitors_THT:C_Rect_L7.0mm_W2.0mm_P5.00mm, symbol ElectricKettle-rescue:C_Small
- removed C? (x2): 100n, Capacitors_THT:C_Rect_L7.0mm_W2.0mm_P5.00mm, symbol ElectricKettle-rescue:C_Small
- removed C?: 100n, symbol device:C
- removed D?: MCU_LED, LEDs:LED_D5.0mm, symbol ElectricKettle-rescue:Led_Small
- removed D? (x4): D, symbol device:D
- removed D?: 1N4001, symbol device:D
- removed D?: 3mm, symbol device:Led_Small
- removed IC?: ATMEGA328-P, Housings_DIP:DIP-28_W7.62mm_LongPads, symbol ElectricKettle-rescue:ATMEGA328-P
- removed P?: FT232_MODULE, Pin_Headers:Pin_Header_Straight_1x06_Pitch1.27mm, symbol ElectricKettle-rescue:CONN_01X06
- removed P?: MAX6675_MODULE, Pin_Headers:Pin_Header_Straight_1x05_Pitch1.27mm, symbol ElectricKettle-rescue:CONN_01X05
- removed P?: ISP_HEADER, symbol conn:CONN_02X03
- removed P?: FLUX_SENSOR, symbol conn:CONN_01X03
- removed P?: ONE_WIRE_SENSOR_1, symbol conn:CONN_01X03
- removed P?: ONE_WIRE_SENSOR_2, symbol conn:CONN_01X03
- removed P?: ONE_WIRE_SENSOR_3, symbol conn:CONN_01X03
- removed R?: 1k2, w_pth_resistors:RC03, symbol ElectricKettle-rescue:R
- removed R?: 470, w_pth_resistors:RC03, symbol ElectricKettle-rescue:R
- removed R?: 100k, w_pth_resistors:RC03, symbol ElectricKettle-rescue:R
- removed R?: 10k, w_pth_resistors:RC03, symbol ElectricKettle-rescue:R
- removed R?: VAR, symbol device:R
- removed R?: 2k7, symbol device:R_Small
- removed R? (x2): R, symbol device:R
- removed SW?: RESET, Buttons_Switches_THT:SW_PUSH_6mm, symbol ElectricKettle-rescue:SW_PUSH_SMALL
- removed U?: DS1302, symbol maxim:DS1302
- removed Y?: 16000, w_pth_resistors:RC03, symbol ElectricKettle-rescue:Crystal_Small
- added D10, D3, D4, D7: 1N4001, Diode_THT:D_DO-35_SOD27_P7.62mm_Horizontal, symbol device:D
- added D11: 1N4001, Diode_THT:D_DO-35_SOD27_P10.16mm_Horizontal, symbol device:D
- added P12, P13: HUM2_SENSOR, TerminalBlock:TerminalBlock_bornier-2_P5.08mm, symbol HUA-rescue:CONN_01X02-conn
- added R12, R13: 1k, Resistor_THT:R_Axial_DIN0207_L6.3mm_D2.5mm_P10.16mm_Horizontal, symbol device:R_Small
- added R14: 20k, Resistor_THT:R_Axial_DIN0207_L6.3mm_D2.5mm_P10.16mm_Horizontal, symbol device:R
- added R15: LDR, Package_TO_SOT_THT:TO-92-2, symbol device:R_PHOTO
- added R20, R21: 100k, Resistor_THT:R_Axial_DIN0207_L6.3mm_D2.5mm_P10.16mm_Horizontal, symbol device:R
- added R22, R23, R24, R26: 1k, Resistor_THT:R_Axial_DIN0207_L6.3mm_D2.5mm_P10.16mm_Horizontal, symbol device:R
- added RV1, RV2, RV3: 20k, Potentiometer_THT:Potentiometer_Bourns_3296W_Vertical, symbol device:R_POT_TRIM
- added U1: NodeMCU_Amica_R2, nodemcu:NodeMCU_Amica_R2, symbol nodemcu:NodeMCU_Amica_R2
- added U3: DS1307+, Package_DIP:DIP-8_W7.62mm_LongPads, symbol Timer_RTC:DS1307+
- added U4: DHT22, Sensors:DHT22_Temperature_Humidity, symbol Sensor:DHT11
- added U5: ADS1115, ADS1115:ADS1115, symbol ADC_MCU_MODULE-cache:ADC_MCU_MODULE-rescue:ADS1115
- BAT1: renamed from BAT?; footprint (none) -> Battery:BatteryHolder_Keystone_106_1x20mm; symbol w_device:BAT -> HUA-rescue:BAT-w_device
- C1, C2, C3, C7, C8: renamed from C?; footprint (none) -> Capacitor_THT:C_Rect_L7.0mm_W2.5mm_P5.00mm
- C4: renamed from C?; footprint Capacitors_THT:C_Rect_L7.0mm_W2.0mm_P5.00mm -> Capacitor_THT:CP_Radial_D10.0mm_P5.00mm; symbol ElectricKettle-rescue:CP -> HUA-rescue:CP-ElectricKettle-rescue
- C5: renamed from C?; footprint Capacitors_THT:CP_Radial_D5.0mm_P2.50mm -> Capacitor_THT:CP_Radial_D5.0mm_P2.50mm; symbol ElectricKettle-rescue:CP -> HUA-rescue:CP-ElectricKettle-rescue
- C6: renamed from C?; footprint (none) -> Capacitor_THT:C_Rect_L7.0mm_W2.5mm_P5.00mm; symbol device:C -> HUA-rescue:C-device
- D1, D2, D6, D8, D9: renamed from D?; footprint (none) -> LED_THT:LED_D3.0mm_Clear; symbol device:Led_Small -> device:LED_Small
- D5: renamed from D?; footprint LEDs:LED_D5.0mm -> LED_THT:LED_D3.0mm; symbol ElectricKettle-rescue:Led_Small -> HUA-rescue:Led_Small-ElectricKettle-rescue
- P1, P10, P2, P5, P6, P9: renamed from P?; footprint (none) -> TerminalBlock:TerminalBlock_bornier-2_P5.08mm; symbol conn:CONN_01X02 -> HUA-rescue:CONN_01X02-conn
- P11: renamed from P?; value HUM_SENSOR -> HUM1_SENSOR; footprint (none) -> TerminalBlock:TerminalBlock_bornier-2_P5.08mm; symbol conn:CONN_01X02 -> HUA-rescue:CONN_01X02-conn
- P3: renamed from P?; value EXT_V3 -> EXT_RL1; footprint (none) -> TerminalBlock:TerminalBlock_bornier-2_P5.08mm; symbol conn:CONN_01X02 -> HUA-rescue:CONN_01X02-conn
- P4: renamed from P?; value VALV_3 -> RL_1; footprint (none) -> TerminalBlock:TerminalBlock_bornier-2_P5.08mm; symbol conn:CONN_01X02 -> HUA-rescue:CONN_01X02-conn
- P7: renamed from P?; value EXT_V3 -> EXT_RL2; footprint (none) -> TerminalBlock:TerminalBlock_bornier-2_P5.08mm; symbol conn:CONN_01X02 -> HUA-rescue:CONN_01X02-conn
- P8: renamed from P?; value VALV_3 -> RL_2; footprint (none) -> TerminalBlock:TerminalBlock_bornier-2_P5.08mm; symbol conn:CONN_01X02 -> HUA-rescue:CONN_01X02-conn
- Q1, Q2, Q3, Q4, Q5: renamed from Q?; footprint TO-92 -> Package_TO_SOT_THT:TO-92_Inline; symbol transistors:BC546 -> HUA-rescue:BC546-transistors
- R1, R2, R5, R8, R9: renamed from R?; value 2k7 -> 1k; footprint (none) -> Resistor_THT:R_Axial_DIN0207_L6.3mm_D2.5mm_P10.16mm_Horizontal
- R10, R11, R3, R4, R7: renamed from R?; footprint (none) -> Resistor_THT:R_Axial_DIN0207_L6.3mm_D2.5mm_P10.16mm_Horizontal; symbol device:R_Small -> HUA-rescue:R_Small-device
- R16, R17, R18: renamed from R?; footprint (none) -> Resistor_THT:R_Axial_DIN0207_L6.3mm_D2.5mm_P10.16mm_Horizontal
- R6: renamed from R?; footprint w_pth_resistors:RC03 -> Resistor_THT:R_Axial_DIN0207_L6.3mm_D2.5mm_P10.16mm_Horizontal; symbol ElectricKettle-rescue:R -> HUA-rescue:R-ElectricKettle-rescue
- RLY1, RLY2, RLY3, RLY4, RLY5: renamed from RLY?; footprint (none) -> Relay_THT:Relay_SPDT_SANYOU_SRD_Series_Form_C; symbol w_relay:RELAY_HJR-3FF_Z -> HUA-rescue:RELAY_HJR-3FF_Z-w_relay
- U2: renamed from U?; footprint TO_SOT_Packages_THT:TO-220_Vertical -> Package_TO_SOT_THT:TO-220-3_Vertical; symbol ElectricKettle-rescue:LM7805CT -> HUA-rescue:LM7805CT-ElectricKettle-rescue
- Y1: renamed from Y?; footprint (none) -> Crystal:Crystal_AT310_D3.0mm_L10.0mm_Vertical
Connections:
- net labels added: +3V3, DHT, HUM1_IN, HUM2_IN, HUM3_IN, LDR
- net labels removed: CTS, DTR, FLUX, HUM_IN, MISO, MOSI, OW_SENSOR1, OW_SENSOR2, OW_SENSOR3, RTC_DATA, RTC_RST, RTC_SCLK, RX, SCK, TX, VCC, XTAL1, XTAL2, ~CS, ~RESET, ~RTC_RST
- wire segments 260 -> 236
- no-connect marks 5 -> 17
Other:
- note added: "MCU INTERFACE\n"
- note added: "RELAY ACTUATOR MODULES\n3 FOR WATER VALVES AND 2 EXTRA FOR LIGHTS\n"
- note added: "SENSOR MODULES\nLIGHT, 3x SOIL HUMIDITY AND ENVIRONMENT TEMP AND HUMIDITY"
- note removed: "FT232 Serial Connections"
- note removed: "MCU INTERFACE\nPULLDOWN SWITCH FOR RESET"
- note removed: "RELAY ACTUATOR MODULES\n3 FOR WATER VALVES AND 2 EXTRA\n"
- note removed: "SENSOR (???) CONNECTIONS\n"
- note removed: "SENSOR MODULES\nWATER FLUX, SOIL HUMIDITY AND 3 EXTRA ONE WIRE SENSORS"
- moved on the sheet: BAT1, C1, C2, C3, C4, C5, C6, C7, C8, D5, P1, P10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

Commit message: ADD: Soil Moisture Sensor circuit and Fabrication Files
Parts:
- removed U5: ADS1115, ADS1115:ADS1115, symbol ADC_MCU_MODULE-cache:ADC_MCU_MODULE-rescue:ADS1115
- added U?: ADC_MCU_MODULE-rescue:ADS1115, symbol ADC_MCU_MODULE-cache:ADC_MCU_MODULE-rescue:ADS1115
- U4: symbol Sensor:DHT11 -> sensors:DHT11
Changed lines of the file:
@@
 EESchema Schematic File Version 4
-LIBS:power
-LIBS:device
-LIBS:transistors
-LIBS:conn
-LIBS:linear
-LIBS:regul
-LIBS:74xx
-LIBS:cmos4000
-LIBS:adc-dac
-LIBS:memory
-LIBS:xilinx
-LIBS:microcontrollers
-LIBS:dsp
-LIBS:microchip
-LIBS:analog_switches
-LIBS:motorola
-LIBS:texas
-LIBS:intel
-LIBS:audio
-LIBS:interface
-LIBS:digital-audio
-LIBS:philips
-LIBS:display
-LIBS:cypress
-LIBS:siliconi
-LIBS:opto
-LIBS:atmel
-LIBS:contrib
-LIBS:valves
 LIBS:HUA-cache
 EELAYER 26 0
@@
 $EndComp
 $Comp
-L Sensor:DHT11 U4
+L sensors:DHT11 U4
 U 1 1 5C1AF8C6
 P 6950 3950
@@
 Wire Wire Line
 	10000 4300 9850 4300
-$Comp
-L ADC_MCU_MODULE-cache:ADC_MCU_MODULE-rescue:ADS1115 U5
-U 1 1 5C8295F4
-P 8650 4550
-F 0 "U5" H 8778 4758 60  0000 L CNN
-F 1 "ADS1115" V 8600 4550 60  0000 L CNN
-F 2 "ADS1115:ADS1115" H 8650 4550 60  0001 C CNN
-F 3 "" H 8650 4550 60  0001 C CNN
-	1    8650 4550
-	1    0    0    -1
-$EndComp
 NoConn ~ 8000 4350
 $Comp
@@
 	0    -1   -1   0
 $EndComp
+$Comp
+L ADC_MCU_MODULE-cache:ADC_MCU_MODULE-rescue:ADS1115 U?
+U 1 1 5C0925F0
+P 8650 4550
+F 0 "U?" H 8777 4758 60  0000 L CNN
+F 1 "ADC_MCU_MODULE-rescue:ADS1115" H 8777 4652 60  0000 L CNN
+F 2 "" H 8650 4550 60  0001 C CNN
+F 3 "" H 8650 4550 60  0001 C CNN
+	1    8650 4550
+	1    0    0    -1
+$EndComp
 $EndSCHEMATC
