File: Eletronica/Soil Moisture Sensor/Soil Moisture Sensor/Soil Moisture Sensor.kicad_pcb (KiCad board)
At the start: 2 copper layers, 21 x 69 mm, 5 parts, among them P1 OUT, U1 NE555

Commit message: EDIT: Soil Moisture Sensor's G-Codes for PCB Milling
Other:
- board size 21 x 69 mm -> 23 x 71.5 mm
- board text added: "G"
- board text added: "S"
- board text added: "V"
Changed lines of the file:
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@@
   (general
     (thickness 1.6)
-    (drawings 15)
+    (drawings 18)
     (tracks 61)
     (zones 0)
@@
     (visible_elements FFFFFF7F)
     (pcbplotparams
-      (layerselection 0x00020_7ffffffe)
+      (layerselection 0x01020_7ffffffe)
       (usegerberextensions false)
       (usegerberattributes false)
@@
       (viasonmask false)
       (mode 1)
-      (useauxorigin false)
+      (useauxorigin true)
       (hpglpennumber 1)
       (hpglpenspeed 20)
@@
       (effects (font (size 1.524 1.524) (thickness 0.3048)))
     )
-    (fp_text value OUT (at 0 4.56946) (layer F.SilkS)
+    (fp_text value OUT (at 0 4.56946) (layer F.SilkS) hide
       (effects (font (size 1.524 1.524) (thickness 0.3048)))
     )
@@
     )
   )
-  (gr_line (start 155.406863 85.756353) (end 155.406863 54.756353) (layer Edge.Cuts) (width 0.15))
-  (gr_line (start 148.406863 85.506353) (end 148.406863 85.756353) (layer Edge.Cuts) (width 0.15))
-  (gr_line (start 148.406863 54.756353) (end 148.406863 85.506353) (layer Edge.Cuts) (width 0.15))
-  (gr_line (start 151.906863 51.256353) (end 148.406863 54.756353) (layer Edge.Cuts) (width 0.15))
-  (gr_line (start 155.406863 54.756353) (end 151.906863 51.256353) (layer Edge.Cuts) (width 0.15))
-  (gr_line (start 134.406863 54.756353) (end 134.406863 120.256353) (layer Edge.Cuts) (width 0.15))
-  (gr_line (start 141.406863 54.756353) (end 141.406863 85.756353) (layer Edge.Cuts) (width 0.15))
-  (gr_line (start 137.906863 51.256353) (end 134.406863 54.756353) (layer Edge.Cuts) (width 0.15))
-  (gr_line (start 141.406863 54.756353) (end 137.906863 51.256353) (layer Edge.Cuts) (width 0.15))
-  (gr_line (start 148.406863 85.756353) (end 141.406863 85.756353) (layer Edge.Cuts) (width 0.15))
-  (gr_line (start 155.406863 85.756353) (end 155.406863 120.256353) (layer Edge.Cuts) (width 0.15))
+  (gr_text G (at 148.906863 119.256353) (layer F.SilkS)
+    (effects (font (size 1.5 1.5) (thickness 0.3)))
+  )
+  (gr_text S (at 146.406863 119.256353) (layer F.SilkS)
+    (effects (font (size 1.5 1.5) (thickness 0.3)))
+  )
+  (gr_text V (at 143.906863 119.256353) (layer F.SilkS)
+    (effects (font (size 1.5 1.5) (thickness 0.3)))
+  )
+  (gr_line (start 156.406863 121.256353) (end 133.406863 121.256353) (layer Edge.Cuts) (width 0.15))
+  (gr_line (start 156.406863 54.256353) (end 156.406863 121.256353) (layer Edge.Cuts) (width 0.15))
+  (gr_line (start 151.906863 49.756353) (end 156.406863 54.256353) (layer Edge.Cuts) (width 0.15))
+  (gr_line (start 147.406863 54.256353) (end 151.906863 49.756353) (layer Edge.Cuts) (width 0.15))
+  (gr_line (start 147.406863 84.756353) (end 147.406863 54.256353) (layer Edge.Cuts) (width 0.15))
+  (gr_line (start 142.406863 84.756353) (end 147.406863 84.756353) (layer Edge.Cuts) (width 0.15))
+  (gr_line (start 142.406863 54.256353) (end 142.406863 84.756353) (layer Edge.Cuts) (width 0.15))
+  (gr_line (start 137.906863 49.756353) (end 142.406863 54.256353) (layer Edge.Cuts) (width 0.15))
+  (gr_line (start 133.406863 54.256353) (end 137.906863 49.756353) (layer Edge.Cuts) (width 0.15))
+  (gr_line (start 133.406863 104.256353) (end 133.406863 54.256353) (layer Edge.Cuts) (width 0.15))
+  (gr_line (start 133.406863 121.256353) (end 133.406863 104.256353) (layer Edge.Cuts) (width 0.2))
+  (gr_line (start 133.406863 104.756353) (end 134.406863 104.756353) (layer F.SilkS) (width 0.2))
+  (gr_line (start 132.406863 104.756353) (end 133.406863 104.756353) (layer F.SilkS) (width 0.2))
   (dimension 7 (width 0.3) (layer Dwgs.User)
     (gr_text "7,000 mm" (at 137.906863 79.156353) (layer Dwgs.User)
@@
     (arrow2b (pts (xy 141.406863 81.256353) (xy 140.280359 81.842774)))
   )
-  (dimension 7 (width 0.3) (layer Dwgs.User)
-    (gr_text "7,000 mm" (at 144.906863 83.656353) (layer Dwgs.User)
-      (effects (font (size 1.5 1.5) (thickness 0.3)))
-    )
-    (feature1 (pts (xy 141.406863 85.756353) (xy 141.406863 85.169932)))
-    (feature2 (pts (xy 148.406863 85.756353) (xy 148.406863 85.169932)))
-    (crossbar (pts (xy 148.406863 85.756353) (xy 141.406863 85.756353)))
-    (arrow1a (pts (xy 141.406863 85.756353) (xy 142.533367 85.169932)))
-    (arrow1b (pts (xy 141.406863 85.756353) (xy 142.533367 86.342774)))
-    (arrow2a (pts (xy 148.406863 85.756353) (xy 147.280359 85.169932)))
-    (arrow2b (pts (xy 148.406863 85.756353) (xy 147.280359 86.342774)))
-  )
-  (gr_line (start 155.406863 120.256353) (end 134.406863 120.256353) (layer Edge.Cuts) (width 0.2))
   (dimension 21 (width 0.3) (layer B.SilkS)
     (gr_text "21,000 mm" (at 144.906863 127.356352) (layer B.SilkS)
